File: hardware/kicad/pcbignicao/pcbignicao/expansao.kicad_sch (KiCad schematic)
At the start: 1 part, among them J12 EXP

Commit message: docs(pcb): adiciona sufixo (THT) aos títulos do projeto de ignição
- Sufixo (THT) nos títulos da raiz e das subfolhas
- Netlist validado: idêntico antes/depois
Other:
- title: Estacao de Ignicao - Expansao -> Estacao de Ignicao (THT) - Expansao
Changed lines of the file:
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@@
 	(paper "A4")
 	(title_block
-		(title "Estacao de Ignicao - Expansao")
+		(title "Estacao de Ignicao (THT) - Expansao")
 		(date "2026-09-23")
 		(rev "1.2")
