File: hardware/kicad/pcbignicao/pcbignicao/interface.kicad_sch (KiCad schematic)
At the start: 10 parts, among them J11 OLED, J3 +buzzer, J4 -buzzer, J5 NO, J9 LED_BTN

Commit message: docs(pcb): adiciona sufixo (THT) aos títulos do projeto de ignição
- Sufixo (THT) nos títulos da raiz e das subfolhas
- Netlist validado: idêntico antes/depois
Other:
- title: Estacao de Ignicao - Interface -> Estacao de Ignicao (THT) - Interface
Changed lines of the file:
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@@
 	(paper "A4")
 	(title_block
-		(title "Estacao de Ignicao - Interface")
+		(title "Estacao de Ignicao (THT) - Interface")
 		(date "2026-09-23")
 		(rev "1.2")
