File: hardware/kicad/pcbignicao/pcbignicao/mcu_pico.kicad_sch (KiCad schematic)
At the start: 1 part

Commit message: docs(pcb): adiciona sufixo (THT) aos títulos do projeto de ignição
- Sufixo (THT) nos títulos da raiz e das subfolhas
- Netlist validado: idêntico antes/depois
Other:
- title: Estacao de Ignicao - MCU_Pico -> Estacao de Ignicao (THT) - MCU_Pico
Changed lines of the file:
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@@
 	(paper "A4")
 	(title_block
-		(title "Estacao de Ignicao - MCU_Pico")
+		(title "Estacao de Ignicao (THT) - MCU_Pico")
 		(date "2026-09-23")
 		(rev "1.2")
