File: hardware/kicad/pcbignicao/pcbignicao/pcbignicao.kicad_sch (KiCad schematic)
At the start: 0 parts

Commit message: docs(pcb): adiciona sufixo (THT) aos títulos do projeto de ignição
- Sufixo (THT) nos títulos da raiz e das subfolhas
- Netlist validado: idêntico antes/depois
Other:
- title: Estacao de Ignicao - LoRa 433 MHz -> Estacao de Ignicao (THT) - LoRa 433 MHz
Changed lines of the file:
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@@
 	(paper "A4")
 	(title_block
-		(title "Estacao de Ignicao - LoRa 433 MHz")
+		(title "Estacao de Ignicao (THT) - LoRa 433 MHz")
 		(date "2026-09-23")
 		(rev "1.2")
