File: hardware/kicad/pcbignicao/pcbignicao/radio_lora.kicad_sch (KiCad schematic)
At the start: 3 parts, among them U1 Ra-02

Commit message: docs(pcb): adiciona sufixo (THT) aos títulos do projeto de ignição
- Sufixo (THT) nos títulos da raiz e das subfolhas
- Netlist validado: idêntico antes/depois
Other:
- title: Estacao de Ignicao - Radio_LoRa -> Estacao de Ignicao (THT) - Radio_LoRa
Changed lines of the file:
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@@
 	(paper "A4")
 	(title_block
-		(title "Estacao de Ignicao - Radio_LoRa")
+		(title "Estacao de Ignicao (THT) - Radio_LoRa")
 		(date "2026-09-23")
 		(rev "1.2")
