File: hardware/kicad/pcbignicao/pcbignicao/saida_ignicao_seguranca.kicad_sch (KiCad schematic)
At the start: 12 parts, among them J10 ARM, J13 SAIDA_IGNICAO, J6 COM, J8 RELE, U2 PC817, U3 PC817

Commit message: docs(pcb): adiciona sufixo (THT) aos títulos do projeto de ignição
- Sufixo (THT) nos títulos da raiz e das subfolhas
- Netlist validado: idêntico antes/depois
Other:
- title: Estacao de Ignicao - Saida_Ignicao_Seguranca -> Estacao de Ignicao (THT) - Saida_Ignicao_Seguranca
Changed lines of the file:
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@@
 	(paper "A4")
 	(title_block
-		(title "Estacao de Ignicao - Saida_Ignicao_Seguranca")
+		(title "Estacao de Ignicao (THT) - Saida_Ignicao_Seguranca")
 		(date "2026-09-23")
 		(rev "1.2")
