File: hardware/kicad/pcbignicao/pcbignicao_smd/interface.kicad_sch (KiCad schematic)
At the start: 10 parts, among them J11 OLED, J3 +buzzer, J4 -buzzer, J5 NO, J9 LED_BTN

Commit message: docs(pcb): normaliza títulos e revisão do projeto SMD
- Sufixo (SMD) nos títulos da raiz e das subfolhas
- Rev 2.0 e data 2026-09-24 alinhados ao README de fabricação
- Corrige comentário que citava a placa THT
- Netlist validado: idêntico antes/depois
Other:
- title: Estacao de Ignicao - Interface -> Estacao de Ignicao (SMD) - Interface
Changed lines of the file:
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@@
 	(paper "A4")
 	(title_block
-		(title "Estacao de Ignicao - Interface")
-		(date "2026-09-23")
-		(rev "1.2")
+		(title "Estacao de Ignicao (SMD) - Interface")
+		(date "2026-09-24")
+		(rev "2.0")
 		(company "Serra Rocketry")
-		(comment 1 "PCB pcbignicao - JLCPCB 2 camadas 1,6 mm - montagem THT manual")
+		(comment 1 "PCB pcbignicao_smd - JLCPCB 2 camadas 1,6 mm - montagem mista (SMD + THT)")
 	)
 	(wire
