File: hardware/kicad/pcbignicao/pcbignicao_smd/mcu_esp32.kicad_sch (KiCad schematic)
At the start: 1 part

Commit message: docs(pcb): normaliza títulos e revisão do projeto SMD
- Sufixo (SMD) nos títulos da raiz e das subfolhas
- Rev 2.0 e data 2026-09-24 alinhados ao README de fabricação
- Corrige comentário que citava a placa THT
- Netlist validado: idêntico antes/depois
Other:
- title: Estacao de Ignicao - MCU (ESP32 NodeMCU-32S) -> Estacao de Ignicao (SMD) - MCU_ESP32
Changed lines of the file:
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@@
 	(paper "A4")
 	(title_block
-		(title "Estacao de Ignicao - MCU (ESP32 NodeMCU-32S)")
+		(title "Estacao de Ignicao (SMD) - MCU_ESP32")
 		(date "2026-09-24")
 		(rev "2.0")
 		(company "Serra Rocketry")
+		(comment 1 "PCB pcbignicao_smd - JLCPCB 2 camadas 1,6 mm - montagem mista (SMD + THT)")
 	)
 	(wire
