File: hardware/kicad/pcbignicao/pcbignicao_smd/radio_lora.kicad_sch (KiCad schematic)
At the start: 3 parts, among them U1 Ra-02

Commit message: docs(pcb): normaliza títulos e revisão do projeto SMD
- Sufixo (SMD) nos títulos da raiz e das subfolhas
- Rev 2.0 e data 2026-09-24 alinhados ao README de fabricação
- Corrige comentário que citava a placa THT
- Netlist validado: idêntico antes/depois
Other:
- title: Estacao de Ignicao - Radio_LoRa -> Estacao de Ignicao (SMD) - Radio_LoRa
Changed lines of the file:
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@@
 	(paper "A4")
 	(title_block
-		(title "Estacao de Ignicao - Radio_LoRa")
-		(date "2026-09-23")
-		(rev "1.2")
+		(title "Estacao de Ignicao (SMD) - Radio_LoRa")
+		(date "2026-09-24")
+		(rev "2.0")
 		(company "Serra Rocketry")
-		(comment 1 "PCB pcbignicao - JLCPCB 2 camadas 1,6 mm - montagem THT manual")
+		(comment 1 "PCB pcbignicao_smd - JLCPCB 2 camadas 1,6 mm - montagem mista (SMD + THT)")
 	)
 	(junction
