File: hardware/kicad/pcbignicao/pcbignicao_smd/saida_ignicao_seguranca.kicad_sch (KiCad schematic)
At the start: 12 parts, among them J10 ARM, J13 SAIDA_IGNICAO, J6 COM, J8 RELE, U2 PC817, U3 PC817

Commit message: feat(pcb): troca U2/U3 de SOP-4 para DIP-4 na ignição SMD (rerroteio pendente)
Parts:
- U2, U3: footprint Package_SO:SOP-4_4.4x2.6mm_P1.27mm -> Package_DIP:DIP-4_W7.62mm_LongPads
Changed lines of the file:
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@@
 			)
 		)
-		(property "Footprint" "Package_SO:SOP-4_4.4x2.6mm_P1.27mm"
+		(property "Footprint" "Package_DIP:DIP-4_W7.62mm_LongPads"
 			(at 231.14 140.97 0)
 			(hide yes)
@@
 			)
 		)
-		(property "Footprint" "Package_SO:SOP-4_4.4x2.6mm_P1.27mm"
+		(property "Footprint" "Package_DIP:DIP-4_W7.62mm_LongPads"
 			(at 231.14 149.86 0)
 			(hide yes)
