File: hardware/kicad/pcbignicao/pcbignicao_smd/pcbignicao_smd.kicad_pcb (KiCad board)
At the start: 2 copper layers, 85 x 70 mm, 36 parts, among them J10 ARM, J11 OLED, J12 EXP, J13 SAIDA_IGNICAO, J3 +buzzer, J4 -buzzer, J5 NO, J6 COM, J7 EXT_PWR, J8 RELE, J9 LED_BTN, U1 Ra-02, U2 PC817, U3 PC817

Commit message: feat(pcb): elimina vias de costura da ignição SMD (rev 2.2)
- Remove as 97 vias de costura restantes; o plano GND fecha com 2 vias de ponte
- Total: 406 -> 24 vias (18 de sinal + 4 GND funcionais + 2 de amarração)
- DRC: 0 itens desconectados e os mesmos 255 avisos de silk/lib (sem regressão)
- Gerbers, drill e pacote JLCPCB regenerados; README e relatório atualizados
Routing:
- net GND: vias 101 -> 6

Commit message: feat(pcb): troca U2/U3 de SOP-4 para DIP-4 na ignição SMD (rerroteio pendente)
Parts:
- U2, U3: footprint SOP-4_4.4x2.6mm_P1.27mm -> DIP-4_W7.62mm_LongPads
Routing:
- net CONT_B: track 51.9 -> 47.0 mm
- net CONT_A: track 76.7 -> 72.0 mm
- net IGN_A: track 47.2 -> 43.7 mm
- net GND: track 20.9 -> 19.6 mm
